File: stereo-mixer/stereo-mixer/preamp-board/preamp-board-v3/preamp-board-v3.kicad_pcb (KiCad board)
At the start: 2 copper layers, 10 parts, among them J1 I/O, U1 LM833N

Commit message: cnc stuff
Parts:
- C3, C4: footprint Capacitor_THT:C_Radial_D5.0mm_H11.0mm_P2.00mm -> Capacitor_THT:C_Radial_D6.3mm_H11.0mm_P2.50mm
- J1: footprint Connector_IDC:IDC-Header_2x20_P2.54mm_Vertical -> Connector_IDC:IDC-Header_2x10_P2.54mm_Vertical
- moved R3 27.1 mm to (354.3, 778.5)
- moved R4 26.7 mm to (354.3, 789.9)
- moved R1 26.7 mm to (354.3, 819.1)
- moved R2 26.7 mm to (354.3, 815.3)
- moved U1 26.7 mm to (354.3, 803.9)
- moved C1 26.7 mm to (359.4, 789.9)
- moved C2 26.7 mm to (359.4, 815.3)
- moved C3 15.9 mm to (312.4, 795.0)
- moved C4 15.9 mm to (318.8, 795.0)
- moved J1 15.9 mm to (328.9, 786.1)
Connections:
- J1 pad 10: Net-(J1-Pad10) -> GND
- J1 pad 12: Net-(J1-Pad12) -> Net-(C1-Pad1)
- J1 pad 13: Net-(C2-Pad1) -> Net-(J1-Pad11)
- J1 pad 15: Net-(C1-Pad1) -> GND
- J1 pad 16: GND -> Net-(C2-Pad1)
- J1 pad 3: Net-(J1-Pad2) -> Net-(J1-Pad3)
- J1 pad 4: GND -> Net-(J1-Pad4)
- J1 pad 5: Net-(C4-Pad1) -> Net-(J1-Pad3)
- J1 pad 7: Net-(J1-Pad6) -> GND
- J1 pad 8: GND -> Net-(J1-Pad8)
- J1 pad 9: Net-(J1-Pad9) -> Net-(C4-Pad1)
- R1 pad 2: Net-(J1-Pad17) -> Net-(J1-Pad8)
- R2 pad 2: Net-(J1-Pad12) -> Net-(J1-Pad18)
- R3 pad 2: Net-(J1-Pad18) -> Net-(J1-Pad6)
- U1 pad 4: Net-(J1-Pad11) -> Net-(J1-Pad20)
- U1 pad 8: Net-(J1-Pad20) -> Net-(J1-Pad2)
Routing:
- net Net-(J1-Pad11): track 109.7 -> 2.54 mm
- net Net-(C2-Pad1): track 182.2 -> 84.2 mm, vias 0 -> 1
- net Net-(C1-Pad1): track 191.8 -> 94.3 mm, vias 0 -> 1
- net Net-(J1-Pad17): track 94.7 -> 0.00 mm
- net Net-(J1-Pad12): track 86.5 -> 0.00 mm
- net Net-(J1-Pad8): track 0.00 -> 68.0 mm
- net Net-(J1-Pad20): track 66.7 -> 23.5 mm
- net Net-(J1-Pad18): track 53.2 -> 19.4 mm
- net Net-(J1-Pad14): track 50.1 -> 21.4 mm, vias 0 -> 1
- net Net-(J1-Pad2): track 12.1 -> 36.5 mm
- net GND: track 100.7 -> 82.2 mm
- net Net-(J1-Pad6): track 30.5 -> 20.5 mm
- net Net-(C1-Pad2): track 20.7 -> 26.2 mm
- net Net-(J1-Pad3): track 0.00 -> 2.54 mm
- net Net-(C4-Pad1): track 11.7 -> 10.7 mm
Other:
- net class Default: via_dia 0.8 -> 2.125; via_drill 0.4 -> 1.5

Commit message: more cnc stuff; sorted out alignment holes
Other:
- board outline added: 101.6 x 69.8 mm
